Commit message: Extended limits

File: simulation/robots/catbot/urdf/catbot.urdf (robot description, URDF)
Before this commit: robot catbot, 13 links, 12 joints
Joints:
- joint LB_0: limit lower=-2 upper=2 effort=1000.0 velocity=1000 -> lower=-6 upper=6 effort=1000.0 velocity=1000
- joint LB_1: limit lower=-2 upper=2 effort=1000.0 velocity=1000 -> lower=-6 upper=6 effort=1000.0 velocity=1000
- joint LB_2: limit lower=-2 upper=2 effort=1000.0 velocity=1000 -> lower=-6 upper=6 effort=1000.0 velocity=1000
- joint LF_1: limit lower=-2 upper=2 effort=1000.0 velocity=1000 -> lower=-6 upper=6 effort=1000.0 velocity=1000
- joint LF_2: limit lower=-2 upper=2 effort=1000.0 velocity=1000 -> lower=-6 upper=6 effort=1000.0 velocity=1000
- joint RB_0: limit lower=-2 upper=2 effort=1000.0 velocity=1000 -> lower=-6 upper=6 effort=1000.0 velocity=1000
- joint RB_1: limit lower=-2 upper=2 effort=1000.0 velocity=1000 -> lower=-6 upper=6 effort=1000.0 velocity=1000
- joint RB_2: limit lower=-2 upper=2 effort=1000.0 velocity=1000 -> lower=-6 upper=6 effort=1000.0 velocity=1000
- joint RF_0: limit lower=-2 upper=2 effort=1000.0 velocity=1000 -> lower=-6 upper=6 effort=1000.0 velocity=1000
- joint RF_1: limit lower=-2 upper=2 effort=1000.0 velocity=1000 -> lower=-6 upper=6 effort=1000.0 velocity=1000
- joint RF_2: limit lower=-2 upper=2 effort=1000.0 velocity=1000 -> lower=-6 upper=6 effort=1000.0 velocity=1000
